Commit message: S20: mobile manipulation platform (LeKiwi + SO-101 + RGB-D cameras)
Mount the SO-101 arm on the LeKiwi mobile base and add the manipulation /
perception layer, a prerequisite for Day 4 (Vision) and Day 5 (Integration).

lekiwi_description:
- mount_link on the deck (empty link; standalone LeKiwi unchanged).
- lekiwi.gazebo.xacro split (lekiwi_gz_plugin / lekiwi_gz_sensors) so the
  platform instantiates a single gz_ros2_control plugin.
- lekiwi.cameras.xacro: two toggleable RGB-D cameras (wrist eye-in-hand + scene).
- lekiwi_manip.urdf.xacro: base + SO-101 arm (arm_ prefix) + cameras,
  gazebo/display/moveit modes, one controller_manager (two ros2_control blocks).

lekiwi_bringup:
- sim_full.launch.py: full sim (base + arm + cameras + EKF + twist_mux).
- ros2_controllers.full.yaml, bridge_full.yaml, arm_initial_positions.yaml.

lekiwi_manipulation_moveit_config: MoveIt 2 for the platform (arm group,
planar virtual joint odom->base_footprint, demo_moveit.launch.py).

lekiwi_manipulation: mobile-manip demo (S20.3) Nav2 navigation -> MoveIt pick
without perception (nav_then_pick + nav_pick_demo.launch.py).

Verified headless: 4 active controllers, RGB-D topics, base<->arm TF, holonomic
teleop, MoveIt arm planning SUCCESS, end-to-end nav->pick demo OK.

Co-Authored-By: Claude Opus 4.8 (1M context) <noreply@anthropic.com>

File: lekiwi_description/urdf/lekiwi.base.xacro (robot description, xacro)
@@ -112,6 +112,13 @@
   </joint>
   <!-- ============================ (S20) mount du bras SO-101 ============ -->
-  <!-- En navigation pure (J2), pas de point de montage du bras.
-       En S20 : ajouter ici un 'mount_link' sur le pont superieur (z ~ ${mount_z})
-       puis include so101_description et fixer arm_base_link a ce frame. -->
+  <!-- Point de montage sur le pont superieur du plateau. Link vide (sans
+       collision/inertie) : inoffensif pour le LeKiwi standalone (navigation J2),
+       et sert d'ancrage au bras SO-101 sur la plateforme de manipulation mobile
+       (cf. lekiwi_manip.urdf.xacro : xacro:so101_arm parent="mount_link"). -->
+  <link name="mount_link"/>
+  <joint name="mount_joint" type="fixed">
+    <parent link="base_link"/>
+    <child link="mount_link"/>
+    <origin xyz="0 0 ${mount_z}" rpy="0 0 0"/>
+  </joint>
 </robot>

File: lekiwi_description/urdf/lekiwi.gazebo.xacro (robot description, xacro)
@@ -2,8 +2,15 @@
 <!-- Integration Gazebo Ionic (gz-sim 9) :
        - plugin gz_ros2_control/GazeboSimSystem (charge controller_manager + controleurs)
-       - capteur gpu_lidar cale sur les specs du LDRobot D500 (360 deg, 720 pts, 0.03-12 m, 10 Hz) -->
+       - capteur gpu_lidar cale sur les specs du LDRobot D500 (360 deg, 720 pts, 0.03-12 m, 10 Hz)
+     Trois macros :
+       lekiwi_gz_plugin(controllers_file) : UNIQUEMENT le plugin gz_ros2_control.
+       lekiwi_gz_sensors()                : frictions roues omni + capteurs IMU/LiDAR.
+       lekiwi_gazebo(controllers_file)    : appelle les deux (LeKiwi standalone, J2).
+     La separation permet a la plateforme de manipulation mobile (LeKiwi + SO-101)
+     de n'instancier QU'UN SEUL plugin gz_ros2_control (un seul controller_manager
+     pour les deux robots) tout en reutilisant les capteurs/frictions du LeKiwi. -->
 <robot xmlns:xacro="http://www.ros.org/wiki/xacro">
-  <xacro:macro name="lekiwi_gazebo" params="controllers_file">
-    <!-- ros2_control via gz_ros2_control -->
+  <!-- ===================== Plugin gz_ros2_control (UN seul par sim) ====== -->
+  <xacro:macro name="lekiwi_gz_plugin" params="controllers_file">
     <gazebo>
       <plugin filename="gz_ros2_control-system"
@@ -12,4 +19,7 @@
       </plugin>
     </gazebo>
+  </xacro:macro>
+  <!-- ===================== Frictions roues omni + capteurs ============== -->
+  <xacro:macro name="lekiwi_gz_sensors">
     <!-- Friction anisotrope des roues omni : traction dans la direction de roulement
          (tangentielle = Y local), glissement libre dans la direction des galets
@@ -66,3 +76,8 @@
     </gazebo>
   </xacro:macro>
+  <!-- ===================== Composite (LeKiwi standalone, J2) ============ -->
+  <xacro:macro name="lekiwi_gazebo" params="controllers_file">
+    <xacro:lekiwi_gz_plugin controllers_file="${controllers_file}"/>
+    <xacro:lekiwi_gz_sensors/>
+  </xacro:macro>
 </robot>
